Commit message: Added ultrasonic sensor data to the navigation.

File: urdf/my_robot.urdf (robot description, URDF)
Before this commit: robot tyler_robot, 6 links, 5 joints
Links:
- added link sonar_link; visual cylinder length=0.0762 radius=0.0254
- link base_link: geometry collision box size=0.81 0.36 0.05; visual box size=0.81 0.36 0.05
Joints:
- added joint sonar_joint: type fixed, parent base_link, child sonar_link, origin xyz=-0.4 0.0 0.015 rpy=0.0 0.0 3.141592653589793
- joint front_left_wheel_joint: origin xyz=0.23 0.2 0 rpy=1.57 0.0 0.0 -> xyz=0.23 0.2 0.025 rpy=1.57 0.0 0.0
- joint front_right_wheel_joint: origin xyz=0.23 -0.2 0 rpy=1.57 0.0 0.0 -> xyz=0.23 -0.2 0.025 rpy=1.57 0.0 0.0
- joint hokuyo_joint: origin xyz=0.4 0.0 -0.01 rpy=0.0 0.0 0.0 -> xyz=0.4 0.0 0.015 rpy=0.0 0.0 3.141592653589793
- joint rear_left_wheel_joint: origin xyz=-0.23 0.2 0 rpy=1.57 0.0 0.0 -> xyz=-0.23 0.2 0.025 rpy=1.57 0.0 0.0
- joint rear_right_wheel_joint: origin xyz=-0.23 -0.2 0 rpy=1.57 0.0 0.0 -> xyz=-0.23 -0.2 0.025 rpy=1.57 0.0 0.0
